File: hardware/MQTT LED.kicad_sch (KiCad schematic)
At the start: 7 parts

Commit message: v1 of the board?
Parts:
- removed Switch: (no value), EasyEDA_Lib:SW-TH_XKB5858-Z-C, symbol EasyEDA_Lib:XKB5858-Z-C
- added C1, C3, C4: 10uF, EasyEDA_Lib:C0805, symbol Device:C
- added C2: 22uF, EasyEDA_Lib:CASE-A_3216, symbol Device:C_Polarized
- added C5: 100nF, EasyEDA_Lib:C0402, symbol Device:C
- added D1: D_Schottky, EasyEDA_Lib:SMBF_L4.3-W3.6-LS5.3-RD, symbol Device:D_Schottky
- added H1, H2, H3, H4: MountingHole, MountingHole:MountingHole_2.1mm, symbol Mechanical:MountingHole
- added L1: 47uH, EasyEDA_Lib:IND-SMD_L8.0-W8.0_ESN8040, symbol Device:L
- added R1, R2: 5.1K, EasyEDA_Lib:R0603, symbol Device:R
- added R3: 100m, EasyEDA_Lib:R1206, symbol Device:R
- J1: renamed from LED-Out; value (none) -> 1x2P; JLC_3DModel_Q (none) -> 3e3e1748db174088b02aeb133ed58c5d; JLC_3D_Size (none) -> 7.5 5.8
- J2: renamed from Flashing/UART; value (none) -> 1x8P; LCSC Part Name 1x8P 间距:2.54mm 方针 直插 -> (none); Manufacturer HanElectricity(瀚源) -> (none); Manufacturer Part 2541WV-08P -> (none); Supplier LCSC -> (none); Supplier Part C5383116 -> (none)
- J3: renamed from Type-C; value (none) -> USB-TYPE-C-009; JLC_3DModel_Q (none) -> ab6076bf4dcb42b58b12fcacb7ccdaa0; JLC_3D_Size (none) -> 8.94 6.8
- U1: renamed from ESP-C2; value (none) -> ESPC2-M1-N2; JLC_3DModel_Q (none) -> 7e1c33b888dd4796bf3789e1a8d334e8; JLC_3D_Size (none) -> 12.3 20
- U2: renamed from LED-Driver; value (none) -> AL8860QMP-13; JLC_3DModel_Q (none) -> a3662aa96ea4496eb423b14219090b21; JLC_3D_Size (none) -> 3 4.9
- U3: renamed from LDO-Regulator; value (none) -> AMS1117-3.3; JLC_3DModel_Q (none) -> e5f8b32b785646b6abbef6d5ae2fe060; JLC_3D_Size (none) -> 7.1095 6.5
Connections:
- net GND: now reaches U3.1 (GND)
- net GND: now also J2.2, J2.5, J3.7 (EH), J3.A12 (GND), J3.B12 (GND), U1.8 (GND), U2.2 (GND), U2.3 (GND), U2.9 (EP), C1.1, C2.2, C3.1, C4.2, C5.2, R1.1, R2.2
- net VBUS: now reaches U3.3 (VIN)
- net VBUS: now also J3.A9 (VBUS), J3.B9 (VBUS), U2.8 (VIN), C1.2, C3.2, D1.1 (K), R3.2
- net +3V3: now reaches U3.4 (VOUT)
- net +3V3: now also U1.7 (VCC), C2.1, C4.1, C5.1
- net BOOT: now reaches U1.10 (IO9)
- net BOOT: now also J2.3
- net EXTRA2: now reaches U1.11 (IO6)
- net EXTRA2: now also J2.4
- net EXTRA1: now reaches U1.12 (IO7)
- net EXTRA1: now also J2.6
- net RX: now reaches U1.13 (RX0)
- net RX: now also J2.7
- net TX: now reaches U1.14 (TX0)
- net TX: now also J2.8
- net RESET: now reaches U1.2 (EN)
- net RESET: now also J2.1
- net CTRL: now reaches U1.9 (IO5)
- net CTRL: now also U2.4 (CTRL)
- net LED+: now reaches U2.1 (SET)
- net LED+: now also J1.1, R3.1
- net at U2.5 (SW): now also U2.6 (SW), D1.2 (A), L1.2
- net LED-: now reaches J1.2
- net LED-: now also L1.1
- net at J3.A5 (CC1): now also R1.2
- net at J3.B5 (CC2): now also R2.1
- no-connect marks 0 -> 8
Other:
- note added: "AL8860QMP-13 LED Driver"
- note added: "AMS1117-3.3 LDO Regulator"
- note added: "ESPC2-M1-N2 MCU Module"
- note added: "IO and LED Pins"
- note added: "Spotlight"
- note added: "USB-C Power Delivery"
- moved on the sheet: J1, J2, J3, U1, U2, U3
